File: Bank-g.kicad_sch (KiCad schematic)
At the start: 1 part, among them U1 XC7K325T-FFG676

Commit message: WIP
WIP - save current state
Parts:
- added D3: LED, LED_SMD:LED_1206_3216Metric_Pad1.42x1.75mm_HandSolder, symbol Device:LED
- added IC11: TXS0108EPWRG4, SamacSys_Parts:SOP65P640X120-20N, symbol SamacSys_Parts:TXS0108EPWRG4
- added IC12: S25FL256LAGMFI001, SamacSys_Parts:SOIC127P1030X265-16N, symbol SamacSys_Parts:S25FL256LAGMFI001
- added J11: Conn_02x05_Odd_Even, Connector_PinHeader_2.54mm:PinHeader_2x05_P2.54mm_Vertical, symbol Connector_Generic:Conn_02x05_Odd_Even
- added J12: Conn_01x06_Socket, Connector_PinSocket_2.54mm:PinSocket_1x06_P2.54mm_Vertical, symbol Connector:Conn_01x06_Socket
- added R65, R66: R, symbol Device:R
- added RN1, RN2, RN3, RN4, RN5: R_Pack04, Resistor_SMD:R_Array_Convex_4x0612, symbol Device:R_Pack04
- added U5, U7: TXS0108EPW, Package_SO:TSSOP-20_4.4x6.5mm_P0.65mm, symbol Logic_LevelTranslator:TXS0108EPW
- added U6: SN74LV245ATPWR, SamacSys_Parts:SOP65P640X120-20N, symbol SamacSys_Parts:SN74LV245ATPWR
Connections:
- net DONE: now reaches U1.J7 (DONE_0)
- net DONE: now also D3.1 (K), R65.1, R66.1
- net GND: now reaches U1.N11 (VREFN_0)
- net GND: now also U1.N12 (VP_0), U1.P11 (VN_0), U1.P12 (VREFP_0), U1.R11 (DXN_0), U1.R12 (DXP_0)
- net VCC_IO: now reaches U1.P7 (CFGBVS_0)
- net VCC_IO: now also D3.2 (A), R65.2, R66.2
Other:
- moved on the sheet: U1G
