File: PCIexpress_x4_half.kicad_pcb (KiCad board)
At the start: 4 copper layers, 167.7 x 111.2 mm, 230 parts, among them IC1 TXS0108EPWRG4, IC10 TMDS141RHAR, IC11 TXS0108EPWRG4, IC12 S25FL256LAGMFI001, IC2 TXS0108EPWRG4, IC3 TPS40057PWP, IC4 TPS54620RHLR, IC5 TPS54620RHLR, IC6 MP2359DJ-LF-Z, IC7 MP2315SGJ-Z, IC8 MP2315SGJ-Z, IC9 TMDS141RHAR, J1 PCIexpress_x4, J10 RJ45_RB1-125B8G1A, J11 Conn_02x05_Odd_Even, J12 Conn_01x06_Socket, J2 PCIexpress_bracket, J3 SFP+, J4 SFP+, J5 2-2013289-2, J6 FAN, J7 Jack-DC, J8 HDMI_A_1.4, J9 HDMI_A_1.4, SW1 SW_SPDT, U1 XC7K325T-FFG676, U3 TPS51200DRC, U4 RTL8211EG-VB-CG, U5 SN74LV245ATPWR, U6 TXS0108EPW, U7 TXS0108EPW, Y1 X32-25.000-12-30_30_4085

Commit message: WIP
Parts:
- added D4: B340, Diode_SMD:D_SMC, F.Cu at (129.1, 74.7)
- added IC13: SI5338A-B04911-GM, SamacSys_Parts:QFN50P400X400X90-25N-D, F.Cu at (135.4, 64.2)
- added U10: XUX53, Oscillator:Oscillator_SMD_IDT_JS6-6_5.0x3.2mm_P1.27mm, F.Cu at (141.4, 51.1)
- added U2: XUX53, Oscillator:Oscillator_SMD_IDT_JS6-6_5.0x3.2mm_P1.27mm, F.Cu at (126.2, 51.1)
- added U8: XUX53, Oscillator:Oscillator_SMD_IDT_JS6-6_5.0x3.2mm_P1.27mm, F.Cu at (131.2, 51.1)
- added U9: XUX53, Oscillator:Oscillator_SMD_IDT_JS6-6_5.0x3.2mm_P1.27mm, F.Cu at (136.3, 51.1)
- added X1: XO91, Oscillator:Oscillator_SMD_EuroQuartz_XO91-4Pin_7.0x5.0mm, F.Cu at (127.9, 64.9)
- added Y2: 25M, Crystal:Crystal_SMD_EuroQuartz_MQ2-2Pin_7.0x5.0mm_HandSoldering, F.Cu at (130.3, 57.7)
Connections:
- IC6 pad 1: unconnected-(IC6-BST-Pad1) -> Net-(IC6-BST)
- IC6 pad 2: unconnected-(IC6-GND-Pad2) -> +12V
- IC6 pad 3: unconnected-(IC6-FB-Pad3) -> Net-(IC6-FB)
- IC6 pad 4: unconnected-(IC6-EN-Pad4) -> Net-(IC6-EN)
- IC6 pad 5: unconnected-(IC6-IN-Pad5) -> Net-(IC6-IN)
- IC6 pad 6: unconnected-(IC6-SW-Pad6) -> Net-(D4-K)
- IC8 pad 1: unconnected-(IC8-AAM-Pad1) -> Net-(IC8-AAM)
- IC8 pad 2: unconnected-(IC8-IN-Pad2) -> +12V
- IC8 pad 3: unconnected-(IC8-SW-Pad3) -> Net-(IC8-SW)
- IC8 pad 4: unconnected-(IC8-GND-Pad4) -> +12V

Commit message: WIP
WIP - save current state
Parts:
- added IC7: MP2315SGJ-Z, SamacSys_Parts:SOT65P280X100-8N, F.Cu at (118.6, 91.0)
- added R46: 27k, Resistor_SMD:R_0201_0603Metric_Pad0.64x0.40mm_HandSolder, F.Cu at (108.9, 89.6)
- added R47: 60k4, Resistor_SMD:R_0201_0603Metric_Pad0.64x0.40mm_HandSolder, F.Cu at (108.9, 91.4)
- added R48: 40k2, Resistor_SMD:R_0201_0603Metric_Pad0.64x0.40mm_HandSolder, F.Cu at (108.9, 93.1)
- added R49: 49k9, Resistor_SMD:R_0201_0603Metric_Pad0.64x0.40mm_HandSolder, F.Cu at (108.9, 94.9)
- added R50: 100k, Resistor_SMD:R_0201_0603Metric_Pad0.64x0.40mm_HandSolder, F.Cu at (108.9, 96.6)
- added R51: 10R, Resistor_SMD:R_0201_0603Metric_Pad0.64x0.40mm_HandSolder, F.Cu at (108.9, 98.4)
- added R52: 100k, Resistor_SMD:R_0201_0603Metric_Pad0.64x0.40mm_HandSolder, F.Cu at (108.9, 100.1)
- added R53: 59k, Resistor_SMD:R_0201_0603Metric_Pad0.64x0.40mm_HandSolder, F.Cu at (111.7, 89.6)
- added R54: 0R, Resistor_SMD:R_0201_0603Metric_Pad0.64x0.40mm_HandSolder, F.Cu at (111.7, 91.4)
- added R55: 40k2, Resistor_SMD:R_0201_0603Metric_Pad0.64x0.40mm_HandSolder, F.Cu at (111.7, 93.1)
- added R56: 31k6, Resistor_SMD:R_0201_0603Metric_Pad0.64x0.40mm_HandSolder, F.Cu at (111.7, 94.9)
- added R57: 53k6, Resistor_SMD:R_0201_0603Metric_Pad0.64x0.40mm_HandSolder, F.Cu at (111.7, 96.6)
- added R58: 47k, Resistor_SMD:R_0201_0603Metric_Pad0.64x0.40mm_HandSolder, F.Cu at (111.7, 98.4)
- added R59: 75k, Resistor_SMD:R_0201_0603Metric_Pad0.64x0.40mm_HandSolder, F.Cu at (111.7, 100.1)
- added R60: 20k5, Resistor_SMD:R_0201_0603Metric_Pad0.64x0.40mm_HandSolder, F.Cu at (114.5, 89.6)
- added R61: 39k2, Resistor_SMD:R_0201_0603Metric_Pad0.64x0.40mm_HandSolder, F.Cu at (114.5, 91.4)
- added R62: 10R, Resistor_SMD:R_0201_0603Metric_Pad0.64x0.40mm_HandSolder, F.Cu at (114.5, 93.1)
- added R63: 0R, Resistor_SMD:R_0201_0603Metric_Pad0.64x0.40mm_HandSolder, F.Cu at (114.5, 94.9)
- added R64: 100k, Resistor_SMD:R_0201_0603Metric_Pad0.64x0.40mm_HandSolder, F.Cu at (114.5, 96.6)
Connections:
- IC8 pad 5: unconnected-(IC8-BST-Pad5) -> Net-(IC8-BST)
- IC8 pad 6: unconnected-(IC8-EN-Pad6) -> Net-(IC8-EN)
- IC8 pad 7: unconnected-(IC8-VCC-Pad7) -> Net-(IC8-VCC)
- IC8 pad 8: unconnected-(IC8-FB-Pad8) -> Net-(IC8-FB)
Routing:
- net /FPGA - kintex/Bank-C/DDR3-B_DQS5-: track 0.00 -> 66.8 mm, vias 0 -> 2
- net /FPGA - kintex/Bank-C/DDR3-B_DQS5+: track 0.00 -> 64.9 mm, vias 0 -> 2
- net /FPGA - kintex/Bank-C/DDR3-B_DQS7+: track 0.00 -> 62.6 mm, vias 0 -> 2
- net /FPGA - kintex/Bank-C/DDR3-B_DQS7-: track 0.00 -> 61.0 mm, vias 0 -> 2
- net /FPGA - kintex/Bank-C/DDR3-B_DQS0-: track 0.00 -> 58.3 mm, vias 0 -> 1
- net /FPGA - kintex/Bank-C/DDR3-B_DQS0+: track 0.00 -> 58.3 mm, vias 0 -> 1
- net /FPGA - kintex/Bank-C/DDR3-B_CLK1-: track 0.00 -> 50.0 mm, vias 0 -> 1
- net /FPGA - kintex/Bank-C/DDR3-B_CLK1+: track 0.00 -> 50.0 mm, vias 0 -> 1
- net /FPGA - kintex/Bank-C/DDR3-B_DQS6+: track 0.00 -> 46.3 mm
- net /FPGA - kintex/Bank-C/DDR3-B_DQS6-: track 0.00 -> 46.0 mm
- net /FPGA - kintex/Bank-C/DDR3-B_DQS1-: track 0.00 -> 42.7 mm
- net /FPGA - kintex/Bank-C/DDR3-B_DQS1+: track 0.00 -> 42.4 mm
- net /FPGA - kintex/Bank-C/DDR3-B_DQS3-: track 0.00 -> 41.6 mm
- net /FPGA - kintex/Bank-C/DDR3-B_DQS3+: track 0.00 -> 41.3 mm
- net /FPGA - kintex/Bank-C/DDR3-B_DQS2-: track 0.00 -> 36.5 mm
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