File: Power.kicad_sch (KiCad schematic)
At the start: 44 parts, among them IC1 TPS40057PWP, J6 FAN, J7 Jack-DC, SW1 SW_SPDT

Commit message: WIP
WIP - save current state
Parts:
- renumbered IC1 to IC3
