File: Power3.kicad_sch (KiCad schematic)
At the start: 3 parts, among them IC6 MP2359DJ-LF-Z, IC7 MP2315SGJ-Z, IC8 MP2315SGJ-Z

Commit message: WIP
Parts:
- added C129: 10n, symbol Device:C
- added C130, C131: 100n, symbol Device:C
- added C132, C133, C134, C135, C142, C144, C146, C147, C148: C, symbol Device:C
- added C136: 22u, symbol Device:C_Polarized
- added C137, C138, C139: 100u, symbol Device:C_Polarized
- added C140, C141, C143, C145: C_Polarized, symbol Device:C_Polarized
- added D4: B340, Diode_SMD:D_SMC, symbol Diode:B340
- added J13: Conn_01x03_Pin, symbol Connector:Conn_01x03_Pin
- added L17, L19: 100n, symbol Device:L
- added L18: L, symbol Device:L
- added L20: 3u5, symbol Device:L_Ferrite
- added L21: L_Ferrite, symbol Device:L_Ferrite
- added L22: 2u2, symbol Device:L_Ferrite
- added R46: 27k, symbol Device:R
- added R47: 60k4, symbol Device:R
- added R48: 40k2, symbol Device:R
- added R49: 49k9, symbol Device:R
- added R50: 100k, symbol Device:R
- added R51, R52, R53, R54, R55, R56, R57, R58, R59, R60, R61, R62, R63, R64: R, symbol Device:R
Connections:
- net at IC8.1 (AAM): now also C132.2, R57.2
- net +12V: now reaches IC8.2 (IN)
- net +12V: now also C140.1
- net at IC8.3 (SW): now also L22.2
- net GND: now reaches IC8.4 (GND)
- net GND: now also IC6.2 (GND), C130.1, C131.1, C132.1, C136.2, C138.2, C139.2, C140.2, R46.2, R47.2, R48.2, R57.1
- net at IC6.1 (BST): now also C129.1
- net at IC6.3 (FB): now also R49.2
- net at IC6.4 (EN): now also R50.2
- net at IC6.5 (IN): now also C130.2, C136.1, R50.1
- net at IC6.6 (SW): now also C129.2, D4.1 (K), L20.1
- new net: C139.1, L19.2, L22.1
- new net: C131.2, C138.1, L19.1
- new net: J13.1 (Pin_1), R46.1
- new net: C137.1, J13.2 (Pin_2), L17.1, L20.2, R48.1, R49.1
- new net: J13.3 (Pin_3), R47.1
- new net: C137.2, D4.2 (A)
- new net VCCIO: L17.2
Other:
- moved on the sheet: IC6, IC8

Commit message: WIP
WIP - save current state
Parts:
- removed C143: C_Polarized, symbol Device:C_Polarized
- removed C144: C, symbol Device:C
- added C143: 1n, symbol Device:C
- added C144: 100u, symbol Device:C_Polarized
- C132: value C -> 1n
- C133, C134, C142, C147, C148: value C -> 100n
- C135, C146: value C -> 22p
- C140, C145: value C_Polarized -> 22u
- C141: value C_Polarized -> 100u
- L18: value L -> 100n
- L21: value L_Ferrite -> 1u5
- R46, R47, R48, R49, R50: footprint (none) -> Resistor_SMD:R_0201_0603Metric_Pad0.64x0.40mm_HandSolder
- R51, R62: value R -> 10R; footprint (none) -> Resistor_SMD:R_0201_0603Metric_Pad0.64x0.40mm_HandSolder
- R52, R64: value R -> 100k; footprint (none) -> Resistor_SMD:R_0201_0603Metric_Pad0.64x0.40mm_HandSolder
- R53: value R -> 59k; footprint (none) -> Resistor_SMD:R_0201_0603Metric_Pad0.64x0.40mm_HandSolder
- R54, R63: value R -> 0R; footprint (none) -> Resistor_SMD:R_0201_0603Metric_Pad0.64x0.40mm_HandSolder
- R55: value R -> 40k2; footprint (none) -> Resistor_SMD:R_0201_0603Metric_Pad0.64x0.40mm_HandSolder
- R56: value R -> 31k6; footprint (none) -> Resistor_SMD:R_0201_0603Metric_Pad0.64x0.40mm_HandSolder
- R57: value R -> 53k6; footprint (none) -> Resistor_SMD:R_0201_0603Metric_Pad0.64x0.40mm_HandSolder
- R58: value R -> 47k; footprint (none) -> Resistor_SMD:R_0201_0603Metric_Pad0.64x0.40mm_HandSolder
- R59: value R -> 75k; footprint (none) -> Resistor_SMD:R_0201_0603Metric_Pad0.64x0.40mm_HandSolder
- R60: value R -> 20k5; footprint (none) -> Resistor_SMD:R_0201_0603Metric_Pad0.64x0.40mm_HandSolder
- R61: value R -> 39k2; footprint (none) -> Resistor_SMD:R_0201_0603Metric_Pad0.64x0.40mm_HandSolder
Connections:
- net +12V: now also C145.1, IC7.2 (IN), R52.1, R64.1
- net GND: now also C133.2, C141.2, C142.1, C145.2, C148.2, IC7.4 (GND), R56.2, R58.1, R61.2, C143.1, C144.2
- net at IC8.3 (SW), L22.2: now also R51.2
- net at IC8.5 (BST): now also C134.1
- net at IC8.6 (EN): now also R52.2
- net at IC8.7 (VCC): now also C133.1
- net at IC8.8 (FB): now also C135.1, R55.1
- net at C139.1, L19.2, L22.1: now also R53.2
- net at C146.1: now also IC7.8 (FB), R60.1
- net at C146.2: now also R63.1
- net at R63.2: now also R59.1, R60.2, R61.1
- net at C135.2: now also R54.1
- net +1V8: now reaches C131.2, C138.1, L19.1
- net +1V2: now reaches C142.2
- net +1V2: now also C141.1, L18.1
- net at C147.1: now also IC7.5 (BST)
- net at C147.2: now also R62.1
- net at IC7.1 (AAM): now also R58.2, C143.2
- net at IC7.3 (SW): now also L21.2, R62.2
- net at IC7.6 (EN): now also R64.2
- net at IC7.7 (VCC): now also C148.1
- net at R59.2: now also L18.2, L21.1, C144.1
- net at R51.1: now also C134.2
- net at R53.1: now also R54.2, R55.2, R56.1
Other:
- moved on the sheet: C133, C134, C135, R52, R54, R55, R56
