File: jtag.kicad_sch (KiCad schematic)
At the start: 13 parts, among them IC11 TXS0108EPWRG4, IC12 S25FL256LAGMFI001, J11 Conn_02x05_Odd_Even, J12 Conn_01x06_Socket, U5 SN74LV245ATPWR, U6 TXS0108EPW, U7 TXS0108EPW

Commit message: WIP
WIP - save current state
Parts:
- removed D3: LED, LED_SMD:LED_1206_3216Metric_Pad1.42x1.75mm_HandSolder, symbol Device:LED
- removed IC11: TXS0108EPWRG4, SamacSys_Parts:SOP65P640X120-20N, symbol SamacSys_Parts:TXS0108EPWRG4
- removed IC12: S25FL256LAGMFI001, SamacSys_Parts:SOIC127P1030X265-16N, symbol SamacSys_Parts:S25FL256LAGMFI001
- removed J11: Conn_02x05_Odd_Even, Connector_PinHeader_2.54mm:PinHeader_2x05_P2.54mm_Vertical, symbol Connector_Generic:Conn_02x05_Odd_Even
- removed J12: Conn_01x06_Socket, Connector_PinSocket_2.54mm:PinSocket_1x06_P2.54mm_Vertical, symbol Connector:Conn_01x06_Socket
- removed RN1, RN2, RN3, RN4, RN5: R_Pack04, Resistor_SMD:R_Array_Convex_4x0612, symbol Device:R_Pack04
- removed U5: SN74LV245ATPWR, SamacSys_Parts:SOP65P640X120-20N, symbol SamacSys_Parts:SN74LV245ATPWR
- removed U6, U7: TXS0108EPW, Package_SO:TSSOP-20_4.4x6.5mm_P0.65mm, symbol Logic_LevelTranslator:TXS0108EPW
